File: eagle/LPC2LCD.brd (EAGLE design)
At the start: 32.4 x 30.4 mm, 8 parts, among them IC1 LC4032V-75TN44C

Commit message: Add files via upload
Connections:
- net 3V3: now also R2.3
- net CONTRAST: no longer R2.1
- net GND: now also R2.1; no longer R2.3
Routing:
- net 3V3: track 56.6 -> 69.0 mm
- net CONTRAST: track 5.75 -> 0.10 mm
- net GND: vias 12 -> 14
Changed lines of the file:
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@@
 <text x="1.143" y="2.794" size="1.016" layer="25" rot="R270">V-</text>
 <text x="15.113" y="24.892" size="0.8128" layer="25" rot="R270">TDO</text>
-<text x="12.573" y="24.765" size="0.8128" layer="25" rot="R270">TDI</text>
-<text x="10.033" y="25.019" size="0.8128" layer="25" rot="R270">TMS</text>
-<text x="7.366" y="25.019" size="0.8128" layer="25" rot="R270">TCK</text>
-<text x="4.953" y="24.765" size="0.8128" layer="25" rot="R270">GND</text>
-<text x="2.286" y="24.638" size="0.8128" layer="25" rot="R270">3v3</text>
+<text x="12.573" y="24.892" size="0.8128" layer="25" rot="R270">TDI</text>
+<text x="10.033" y="24.892" size="0.8128" layer="25" rot="R270">TMS</text>
+<text x="7.366" y="24.892" size="0.8128" layer="25" rot="R270">TCK</text>
+<text x="4.953" y="24.892" size="0.8128" layer="25" rot="R270">GND</text>
+<text x="2.286" y="24.892" size="0.8128" layer="25" rot="R270">3v3</text>
 <wire x1="-0.254" y1="28.956" x2="-0.254" y2="1.524" width="0.3048" layer="20"/>
 <wire x1="-0.254" y1="1.524" x2="1.27" y2="0" width="0.3048" layer="20"/>
@@
 <attribute name="MOUSER_PRICE-STOCK" value="https://www.mouser.com/Search/Refine.aspx?Keyword=842-LC4032V75TN44C" x="19.304" y="37.084" size="1.778" layer="27" rot="R90" display="off"/>
 <attribute name="NAME" x="9.144" y="14.224" size="1.27" layer="25" rot="R180" align="center"/>
-<attribute name="VALUE" x="-39.116" y="19.304" size="1.27" layer="27" rot="R90" align="center"/>
 </element>
 <element name="LPC" library="con-lstb" library_urn="urn:adsk.eagle:library:162" package="MA06-2" package3d_urn="urn:adsk.eagle:package:8342/1" value="" x="26.797" y="16.002" smashed="yes" rot="R90">
@@
 <signal name="RST">
 <contactref element="IC1" pad="18"/>
-<wire x1="26" y1="16.25" x2="17.5" y2="16.25" width="0.1524" layer="1"/>
-<wire x1="27.5" y1="14.75" x2="26" y2="16.25" width="0.1524" layer="1"/>
+<wire x1="26.127" y1="16.123" x2="17.7251375" y2="16.123" width="0.1524" layer="1"/>
+<wire x1="27.5" y1="14.75" x2="26.127" y2="16.123" width="0.1524" layer="1"/>
 <wire x1="28" y1="14.75" x2="27.5" y2="14.75" width="0.1524" layer="1"/>
-<wire x1="17.5" y1="16.25" x2="17.422" y2="16.294" width="0.1524" layer="1"/>
+<wire x1="17.7251375" y1="16.123" x2="17.422" y2="16.294" width="0.1524" layer="1"/>
 <contactref element="LPC" pad="5"/>
 <wire x1="28.0416" y1="14.7828" x2="28.067" y2="14.732" width="0.1524" layer="1"/>
@@
 <wire x1="7.75" y1="21" x2="7.684" y2="21.232" width="0.1524" layer="1"/>
 <wire x1="11.5" y1="21" x2="11.684" y2="21.232" width="0.1524" layer="1"/>
-<wire x1="2.5" y1="26.25" x2="7.5" y2="21.25" width="0.1524" layer="1"/>
+<wire x1="2.5" y1="26.25" x2="7.5" y2="21.25" width="0.3048" layer="1"/>
 <wire x1="7.5" y1="21.25" x2="7.684" y2="21.232" width="0.1524" layer="1"/>
 <wire x1="11.75" y1="19.75" x2="11.75" y2="12.528" width="0.3048" layer="1"/>
@@
 <contactref element="JP1" pad="1"/>
 <wire x1="2.5" y1="26.25" x2="2.667" y2="26.289" width="0.1524" layer="1"/>
+<contactref element="R2" pad="3"/>
+<wire x1="7.684" y1="21.232" x2="6.21515" y2="21.232" width="0.3048" layer="1"/>
+<wire x1="6.21515" y1="21.232" x2="5.83935" y2="20.8562" width="0.3048" layer="1"/>
+<wire x1="5.83935" y1="20.8562" x2="4.9812" y2="20.8562" width="0.3048" layer="1"/>
+<wire x1="2.54" y1="18.415" x2="2.54" y2="12.293" width="0.3048" layer="1"/>
+<wire x1="4.9812" y1="20.8562" x2="2.54" y2="18.415" width="0.3048" layer="1"/>
 </signal>
 <signal name="LAD0">
@@
 <contactref element="LPC" pad="10"/>
 <contactref element="IC1" pad="21"/>
-<wire x1="23.25" y1="18.75" x2="17.5" y2="18.75" width="0.1524" layer="1"/>
-<wire x1="24.25" y1="19.75" x2="23.25" y2="18.75" width="0.1524" layer="1"/>
-<wire x1="25.5" y1="19.75" x2="24.25" y2="19.75" width="0.1524" layer="1"/>
-<wire x1="17.5" y1="18.75" x2="17.422" y2="18.694" width="0.1524" layer="1"/>
-<wire x1="25.5" y1="19.75" x2="25.527" y2="19.812" width="0.1524" layer="1"/>
+<wire x1="21.98" y1="18.75" x2="17.478" y2="18.75" width="0.1524" layer="1"/>
+<wire x1="17.422" y1="18.694" x2="17.478" y2="18.75" width="0.1524" layer="1"/>
+<wire x1="22.599" y1="19.369" x2="21.98" y2="18.75" width="0.1524" layer="1"/>
+<wire x1="25.33408125" y1="19.369" x2="22.599" y2="19.369" width="0.1524" layer="1"/>
+<wire x1="25.33408125" y1="19.369" x2="25.527" y2="19.812" width="0.1524" layer="1"/>
 </signal>
 <signal name="LAD2">
@@
 <wire x1="11" y1="9.75" x2="10.884" y2="9.756" width="0.1524" layer="1"/>
 <wire x1="11" y1="9.75" x2="10.907" y2="9.77901875" width="0.1524" layer="1"/>
-<via x="10.287" y="16.637" extent="1-16" drill="0.35"/>
+<via x="9.398" y="17.526" extent="1-16" drill="0.35"/>
 <via x="13.97" y="15.875" extent="1-16" drill="0.35"/>
 <via x="5.588" y="21.463" extent="1-16" drill="0.35"/>
-<contactref element="R2" pad="3"/>
 <via x="10.668" y="7.747" extent="1-16" drill="0.3"/>
 <via x="11.811" y="8.382" extent="1-16" drill="0.3"/>
@@
 <via x="16.002" y="6.731" extent="1-16" drill="0.3"/>
 <via x="5.334" y="7.747" extent="1-16" drill="0.3"/>
-<via x="22.733" y="14.859" extent="1-16" drill="0.3"/>
+<via x="23.241" y="14.986" extent="1-16" drill="0.3"/>
 <via x="22.606" y="19.939" extent="1-16" drill="0.3"/>
 <contactref element="JP1" pad="2"/>
@@
 <contactref element="JP2" pad="12"/>
 <contactref element="JP2" pad="5"/>
+<via x="22.606" y="18.542" extent="1-16" drill="0.3"/>
+<via x="22.987" y="16.637" extent="1-16" drill="0.3"/>
+<contactref element="R2" pad="1"/>
 </signal>
 <signal name="TCK">
@@
 <contactref element="IC1" pad="32"/>
 <contactref element="JP1" pad="6"/>
-<via x="13.335" y="22.86" extent="1-16" drill="0.35"/>
+<via x="14.351" y="23.241" extent="1-16" drill="0.35"/>
 <wire x1="8.484" y1="21.232" x2="8.7554" y2="21.5034" width="0.1524" layer="1"/>
 <wire x1="8.7554" y1="21.5034" x2="8.7554" y2="22.0641875" width="0.1524" layer="1"/>
-<wire x1="8.7554" y1="22.0641875" x2="9.5512125" y2="22.86" width="0.1524" layer="1"/>
-<wire x1="9.5512125" y1="22.86" x2="13.335" y2="22.86" width="0.1524" layer="1"/>
-<wire x1="13.335" y1="22.86" x2="15.367" y2="24.892" width="0.1524" layer="16"/>
-<wire x1="15.367" y1="24.892" x2="15.367" y2="26.289" width="0.1524" layer="16"/>
+<wire x1="8.7554" y1="22.0641875" x2="9.8052125" y2="23.114" width="0.1524" layer="1"/>
+<wire x1="14.224" y1="23.114" x2="14.351" y2="23.241" width="0.1524" layer="1"/>
+<wire x1="14.224" y1="23.114" x2="9.8052125" y2="23.114" width="0.1524" layer="1"/>
+<wire x1="14.351" y1="23.241" x2="15.367" y2="24.257" width="0.1524" layer="16"/>
+<wire x1="15.367" y1="24.257" x2="15.367" y2="26.289" width="0.1524" layer="16"/>
 </signal>
 <signal name="N$1">
@@
 <signal name="CONTRAST">
 <contactref element="IC1" pad="43"/>
-<contactref element="R2" pad="1"/>
-<wire x1="5.0292" y1="12.192" x2="2.170371875" y2="9.333171875" width="0.1524" layer="1"/>
-<wire x1="5.9436" y1="12.192" x2="5.0292" y2="12.192" width="0.1524" layer="1"/>
-<wire x1="2.170371875" y1="9.333171875" x2="1.54" y2="9.043" width="0.1524" layer="1"/>
 <wire x1="5.9436" y1="12.192" x2="5.946" y2="12.294" width="0.1524" layer="1"/>
 </signal>
